Commit message: change

File: quadruped_robot/urdf/spotmicroai_gen_ros.xacro (robot description, xacro)
@@ -608,3 +608,135 @@
     <origin xyz="0 0 -0.115"/>
   </joint>
+    <!-- ros2_control block -->
+  <ros2_control>
+    <hardware>
+      <plugin>QuadrupedDynamixelHardware</plugin>
+      <param name="usb_port">/dev/ttyUSB0</param>
+      <param name="baud_rate">57600</param>
+    </hardware>
+  </ros2_control>
+<!-- Transmissions for front left leg -->
+<transmission name="front_left_hip_trans">
+  <type>SimpleTransmission</type>
+  <joint name="front_left_hip_joint">
+    <hardwareInterface>hardware_interface/PositionJointInterface</hardwareInterface>
+  </joint>
+  <actuator name="front_left_hip_motor">
+    <hardwareInterface>hardware_interface/PositionJointInterface</hardwareInterface>
+    <mechanicalReduction>1</mechanicalReduction>
+  </actuator>
+</transmission>
+<transmission name="front_left_knee_trans">
+  <type>SimpleTransmission</type>
+  <joint name="front_left_knee_joint">
+    <hardwareInterface>hardware_interface/PositionJointInterface</hardwareInterface>
+  </joint>
+  <actuator name="front_left_knee_motor">
+    <hardwareInterface>hardware_interface/PositionJointInterface</hardwareInterface>
+    <mechanicalReduction>1</mechanicalReduction>
+  </actuator>
+</transmission>
+<transmission name="front_left_ankle_trans">
+  <type>SimpleTransmission</type>
+  <joint name="front_left_ankle_joint">
+    <hardwareInterface>hardware_interface/PositionJointInterface</hardwareInterface>
+  </joint>
+  <actuator name="front_left_ankle_motor">
+    <hardwareInterface>hardware_interface/PositionJointInterface</hardwareInterface>
+    <mechanicalReduction>1</mechanicalReduction>
+  </actuator>
+</transmission>
+<!-- Transmissions for front right leg -->
+<transmission name="front_right_hip_trans">
+  <type>SimpleTransmission</type>
+  <joint name="front_right_hip_joint">
+    <hardwareInterface>hardware_interface/PositionJointInterface</hardwareInterface>
+  </joint>
+  <actuator name="front_right_hip_motor">
+    <hardwareInterface>hardware_interface/PositionJointInterface</hardwareInterface>
+    <mechanicalReduction>1</mechanicalReduction>
+  </actuator>
+</transmission>
+<transmission name="front_right_knee_trans">
+  <type>SimpleTransmission</type>
+  <joint name="front_right_knee_joint">
+    <hardwareInterface>hardware_interface/PositionJointInterface</hardwareInterface>
+  </joint>
+  <actuator name="front_right_knee_motor">
+    <hardwareInterface>hardware_interface/PositionJointInterface</hardwareInterface>
+    <mechanicalReduction>1</mechanicalReduction>
+  </actuator>
+</transmission>
+<transmission name="front_right_ankle_trans">
+  <type>SimpleTransmission</type>
+  <joint name="front_right_ankle_joint">
+    <hardwareInterface>hardware_interface/PositionJointInterface</hardwareInterface>
+  </joint>
+  <actuator name="front_right_ankle_motor">
+    <hardwareInterface>hardware_interface/PositionJointInterface</hardwareInterface>
+    <mechanicalReduction>1</mechanicalReduction>
+  </actuator>
+</transmission>
+<!-- Transmissions for rear left leg -->
+<transmission name="rear_left_hip_trans">
+  <type>SimpleTransmission</type>
+  <joint name="rear_left_hip_joint">
+    <hardwareInterface>hardware_interface/PositionJointInterface</hardwareInterface>
+  </joint>
+  <actuator name="rear_left_hip_motor">
+    <hardwareInterface>hardware_interface/PositionJointInterface</hardwareInterface>
+    <mechanicalReduction>1</mechanicalReduction>
+  </actuator>
+</transmission>
+<transmission name="rear_left_knee_trans">
+  <type>SimpleTransmission</type>
+  <joint name="rear_left_knee_joint">
+    <hardwareInterface>hardware_interface/PositionJointInterface</hardwareInterface>
+  </joint>
+  <actuator name="rear_left_knee_motor">
+    <hardwareInterface>hardware_interface/PositionJointInterface</hardwareInterface>
+    <mechanicalReduction>1</mechanicalReduction>
+  </actuator>
+</transmission>
+<transmission name="rear_left_ankle_trans">
+  <type>SimpleTransmission</type>
+  <joint name="rear_left_ankle_joint">
+    <hardwareInterface>hardware_interface/PositionJointInterface</hardwareInterface>
+  </joint>
+  <actuator name="rear_left_ankle_motor">
+    <hardwareInterface>hardware_interface/PositionJointInterface</hardwareInterface>
+    <mechanicalReduction>1</mechanicalReduction>
+  </actuator>
+</transmission>
+<!-- Transmissions for rear right leg -->
+<transmission name="rear_right_hip_trans">
+  <type>SimpleTransmission</type>
+  <joint name="rear_right_hip_joint">
+    <hardwareInterface>hardware_interface/PositionJointInterface</hardwareInterface>
+  </joint>
+  <actuator name="rear_right_hip_motor">
+    <hardwareInterface>hardware_interface/PositionJointInterface</hardwareInterface>
+    <mechanicalReduction>1</mechanicalReduction>
+  </actuator>
+</transmission>
+<transmission name="rear_right_knee_trans">
+  <type>SimpleTransmission</type>
+  <joint name="rear_right_knee_joint">
+    <hardwareInterface>hardware_interface/PositionJointInterface</hardwareInterface>
+  </joint>
+  <actuator name="rear_right_knee_motor">
+    <hardwareInterface>hardware_interface/PositionJointInterface</hardwareInterface>
+    <mechanicalReduction>1</mechanicalReduction>
+  </actuator>
+</transmission>
+<transmission name="rear_right_ankle_trans">
+  <type>SimpleTransmission</type>
+  <joint name="rear_right_ankle_joint">
+    <hardwareInterface>hardware_interface/PositionJointInterface</hardwareInterface>
+  </joint>
+  <actuator name="rear_right_ankle_motor">
+    <hardwareInterface>hardware_interface/PositionJointInterface</hardwareInterface>
+    <mechanicalReduction>1</mechanicalReduction>
+  </actuator>
+</transmission>
 </robot>
