Commit message: added spot/champ final file

File: quadruped_robot/urdf/spot.urdf.xacro (robot description, xacro)
@@ -1,100 +1,935 @@
-<?xml version="1.0"?>
-<robot xmlns:xacro="http://www.ros.org/wiki/xacro" name="spot">
-  <xacro:property name="wheel_radius" value="0.03"/>
-  <xacro:property name="wheel_separation" value="0.335"/>
-  <xacro:property name="caster_wheel_radius" value="${wheel_radius/2}"/>
-  <xacro:property name="caster_wheel_mass" value="0.001"/>
-  <xacro:property name="caster_wheel_joint_offset" value="0.3"/>
-  <xacro:property name="wheel_offset" value="0.025"/>
-  <xacro:macro name="default_inertial" params="mass">
-    <inertial>
-      <mass value="${mass}"/>
-      <inertia ixx="1.0" ixy="0.0" ixz="0.0" iyy="1.0" iyz="0.0" izz="1.0"/>
-    </inertial>
-  </xacro:macro>
-  <xacro:macro name="cylinder_inertia" params="m r h">
-    <inertial>
-      <mass value="${m}"/>
-      <inertia ixx="${m*(3*r*r+h*h)/12}" ixy = "0" ixz = "0" iyy="${m*(3*r*r+h*h)/12}" iyz = "0" izz="${m*r*r/2}"/>
-    </inertial>
-  </xacro:macro>
-  <!-- not used currently but maybe can be used for better spot model inertia estimation
-    <xacro:macro name="box_inertia" params="m w h d">
-    <inertial>
-      <mass value="${m}"/>
-      <inertia ixx="${m / 12.0 * (d*d + h*h)}" ixy="0.0" ixz="0.0" iyy="${m / 12.0 * (w*w + h*h)}" iyz="0.0" izz="${m / 12.0 * (w*w + d*d)}"/>
-    </inertial>
-  </xacro:macro> -->
-  <xacro:macro name="sphere_inertia" params="m r">
-    <inertial>
-      <mass value="${m}"/>
-      <inertia ixx="${2.0*m*(r*r)/5.0}" ixy="0.0" ixz="0.0" iyy="${2.0*m*(r*r)/5.0}" iyz="0.0" izz="${2.0*m*(r*r)/5.0}"/>
-    </inertial>
-  </xacro:macro>
-  <!-- <link name="base_footprint" />
-  <joint name="footprint" type="fixed" >
-    <parent link="base_footprint" />
-    <child link="base_footprint" />
-    <origin xyz="0 0 0.655" rpy="0 0 0" />
-  </joint> -->
-  <link name="base_footprint">
-    <xacro:default_inertial mass="32.5"/>
-    <visual name="visual">
-      <origin xyz="0 0 0.655" rpy="0 0 0" />
-      <geometry>
-        <mesh filename="package://quadruped_robot/meshes/spot_whole_body.dae" />
-      </geometry>
-    </visual>
-    <collision>
-      <origin xyz="0 0 0.655" rpy="0 0 0" />
-      <geometry>
-        <mesh filename="package://quadruped_robot/meshes/spot_whole_body.dae" />
-      </geometry>
-    </collision>
-  </link>
-  <xacro:macro name="wheel" params="prefix reflect">
-    <link name="${prefix}_wheel">
-      <collision>
-        <origin xyz="0 0 0" rpy="${pi/2} 0 0"/>
-        <geometry>
-          <cylinder radius="${wheel_radius}" length="0.005"/>
-        </geometry>
-      </collision>
-      <xacro:cylinder_inertia m="0.5" r="${wheel_radius}" h="0.005"/>
-    </link>
-    <joint name="${prefix}_wheel_joint" type="continuous">
-      <axis xyz="0 1 0" rpy="0 0 0" />
-      <parent link="base_footprint"/>
-      <child link="${prefix}_wheel"/>
-      <origin xyz="${wheel_offset} ${(wheel_separation/2)*reflect} -0.005" rpy="0 0 0"/>
-    </joint>
-  </xacro:macro>
-  <xacro:wheel prefix="left" reflect="0.6"/>
-  <xacro:wheel prefix="right" reflect="-0.6"/>
-  <xacro:macro name="caster" params="prefix reflectH reflectV">
-    <link name="${prefix}_caster_wheel">
-      <collision>
-        <origin xyz="0 0 0" rpy="0 0 0"/>
-        <geometry>
-          <sphere radius="${caster_wheel_radius}"/>
-        </geometry>
-      </collision>
-      <xacro:sphere_inertia m="0.05" r="${caster_wheel_radius}"/>
-    </link>
-    <joint name="${prefix}_caster_wheel_joint" type="continuous">
-      <axis xyz="0 1 0" rpy="0 0 0" />
-      <parent link="base_footprint"/>
-      <child link="${prefix}_caster_wheel"/>
-      <origin xyz="${wheel_offset + caster_wheel_joint_offset*reflectV} ${wheel_separation/2*reflectH} -${caster_wheel_radius+0.005}" rpy="0 0 0"/>
-    </joint>
-  </xacro:macro>
-  <!-- <xacro:caster prefix="front_left" reflectH="1" reflectV="1"/>
-  <xacro:caster prefix="front_right" reflectH="-1" reflectV="1"/> -->
-  <xacro:caster prefix="back_left" reflectH="1" reflectV="-1"/>
-  <xacro:caster prefix="back_right" reflectH="-1" reflectV="-1"/>
-  <!-- <xacro:include filename="$(find quadruped_robot)/urdf/spot.plugins.xacro"/> -->
-  <!-- <xacro:include filename="$(find velodyne_description)/urdf/VLP-16.urdf.xacro"/> -->
-  <!-- <xacro:VLP-16 parent="base_footprint" name="velodyne" topic="/lidar_points" hz="10" samples="1024" gpu="false" lasers="16" max_range="100">
-    <origin xyz="0 0 0.73" rpy="0 0 0" />
-  </xacro:VLP-16> -->
+<?xml version="1.0" ?>
+<robot name="spotmicroai">
+  <!-- Params -->
+  <!-- Macros -->
+  <!-- Robot Body -->
+  <!--test-->
+  <link name="base_link">
+    <visual>
+      <geometry>
+        <mesh filename="file://$(find quadruped_robot)/stl/mainbody.stl" scale="0.001 0.001 0.001"/>
+      </geometry>
+      <origin rpy="0 0 0" xyz="-0.045 -0.060 -0.015"/>
+      <material name="black">
+        <color rgba="0.0 0.0 0.0 1.0"/>
+      </material>
+    </visual>
+    <collision>
+      <geometry>
+        <mesh filename="file://$(find quadruped_robot)/stl/mainbody.stl" scale="0.001 0.001 0.001"/>
+      </geometry>
+      <origin rpy="0 0 0" xyz="-0.045 -0.060 -0.015"/>
+    </collision>
+    <inertial>
+        <mass value="2.0"/> <!-- Approximate base mass in kg -->
+        <origin xyz="0.0 0.0 0.0" rpy="0 0 0"/> <!-- Adjust center of mass -->
+        <inertia
+            ixx="0.007"
+            ixy="0.0"
+            ixz="0.0"
+            iyy="0.008"
+            iyz="0.0"
+            izz="0.009"/>
+    </inertial>
+  </link>
+  <!-- Lidar Backpack -->
+  <link name="lidar_link">
+    <visual>
+      <geometry>
+        <mesh filename="file://$(find quadruped_robot)/stl/rplidar_main.STL" scale="0.001 0.001 0.001"/>
+      </geometry>
+      <material name="black"/>
+      <origin rpy="1.57075 0 0" xyz="-0.06425 0.02885 0"/>
+    </visual>
+    <collision>
+      <geometry>
+        <mesh filename="file://$(find quadruped_robot)/stl/rplidar_main.STL" scale="0.001 0.001 0.001"/>
+      </geometry>
+      <origin rpy="1.57075 0 0" xyz="-0.06425 0.02885 0"/>
+    </collision>
+    <inertial>
+      <mass value="0.02"/>
+      <inertia ixx="0.05" ixy="0" ixz="0" iyy="0.05" iyz="0" izz="0.05"/>
+    </inertial>
+  </link>
+  <joint name="base_lidar" type="fixed">
+    <parent link="base_link"/>
+    <child link="lidar_link"/>
+    <origin xyz="0 0 0.035"/>
+  </joint>
+  <link name="rear_link">
+    <visual>
+      <geometry>
+        <mesh filename="file://$(find quadruped_robot)/stl/backpart.stl" scale="0.001 0.001 0.001"/>
+      </geometry>
+      <origin rpy="0 0 0" xyz="-0.040 -0.060 -0.0140"/>
+      <material name="yellow">
+        <color rgba="0.92 0.83 0.0 1"/>
+      </material>
+    </visual>
+    <collision>
+      <geometry>
+        <mesh filename="file://$(find quadruped_robot)/stl/backpart.stl" scale="0.001 0.001 0.001"/>
+      </geometry>
+      <origin rpy="0 0 0" xyz="-0.040 -0.060 -0.0140"/>
+    </collision>
+    <inertial>
+      <mass value="0.20"/>
+      <inertia ixx="0.05" ixy="0" ixz="0" iyy="0.05" iyz="0" izz="0.05"/>
+    </inertial>
+  </link>
+  <joint name="base_rear" type="fixed">
+    <parent link="base_link"/>
+    <child link="rear_link"/>
+  </joint>
+  <link name="front_link">
+    <visual>
+      <geometry>
+        <mesh filename="file://$(find quadruped_robot)/stl/frontpart.stl" scale="0.001 0.001 0.001"/>
+      </geometry>
+      <origin rpy="0 0 0" xyz="-0.040 -0.060 -0.0140"/>
+      <material name="yellow">
+        <color rgba="0.92 0.83 0.0 1"/>
+      </material>
+    </visual>
+    <collision>
+      <geometry>
+        <mesh filename="file://$(find quadruped_robot)/stl/frontpart.stl" scale="0.001 0.001 0.001"/>
+      </geometry>
+      <origin rpy="0 0 0" xyz="-0.040 -0.060 -0.0140"/>
+    </collision>
+    <inertial>
+      <mass value="0.20"/>
+      <inertia ixx="0.05" ixy="0" ixz="0" iyy="0.05" iyz="0" izz="0.05"/>
+    </inertial>
+  </link>
+  <joint name="base_front" type="fixed">
+    <parent link="base_link"/>
+    <child link="front_link"/>
+  </joint>
+  <link name="imu_link">
+    <inertial>
+      <mass value="0.01"/>
+      <origin rpy="0 0 0" xyz="0 0 0"/>
+      <inertia ixx="0.0001" ixy="0" ixz="0" iyy="0.0001" iyz="0" izz="0.0001"/>
+    </inertial>
+  </link>
+  <joint name="imu_joint" type="fixed">
+    <parent link="base_link"/>
+    <child link="imu_link"/>
+    <origin rpy="0 0 0" xyz="0 0 0"/>
+  </joint>
+  <!-- create Legs -->
+  <link name="front_left_shoulder_link">
+    <visual>
+      <geometry>
+        <mesh filename="file://$(find quadruped_robot)/stl/lshoulder.stl" scale="0.001 0.001 0.001"/>
+      </geometry>
+      <origin rpy="0 0 0" xyz="-0.135 -0.02 -0.01"/>
+      <material name="black">
+        <color rgba="0.0 0.0 0.0 1.0"/>
+      </material>
+    </visual>
+    <collision>
+      <geometry>
+        <mesh filename="file://$(find quadruped_robot)/stl/lshoulder.stl" scale="0.001 0.001 0.001"/>
+      </geometry>
+      <origin rpy="0 0 0" xyz="-0.135 -0.02 -0.01"/>
+    </collision>
+    <inertial>
+      <mass value="0.30"/>
+      <inertia ixx="0.0005" ixy="0" ixz="0" iyy="0.0006" iyz="0" izz="0.0007"/>
+    </inertial>
+  </link>
+  <link name="front_left_leg_link_cover">
+    <visual>
+      <geometry>
+        <mesh filename="file://$(find quadruped_robot)/stl/larm_cover.stl" scale="0.001 0.001 0.001"/>
+      </geometry>
+      <origin rpy="0 0 0" xyz="-0.125 0.04 -0.02"/>
+      <material name="yellow">
+        <color rgba="0.92 0.83 0.0 1"/>
+      </material>
+    </visual>
+  </link>
+  <link name="front_left_leg_link">
+    <visual>
+      <geometry>
+        <mesh filename="file://$(find quadruped_robot)/stl/larm.stl" scale="0.001 0.001 0.001"/>
+      </geometry>
+      <origin rpy="0 0 0" xyz="-0.125 0.04 -0.02"/>
+      <material name="black">
+        <color rgba="0.0 0.0 0.0 1.0"/>
+      </material>
+    </visual>
+    <collision>
+      <geometry>
+        <mesh filename="file://$(find quadruped_robot)/stl/larm.stl" scale="0.001 0.001 0.001"/>
+      </geometry>
+      <origin rpy="0 0 0" xyz="-0.125 0.04 -0.02"/>
+    </collision>
+    <inertial>
+      <mass value="0.2"/>
+      <inertia ixx="0.0002" ixy="0" ixz="0" iyy="0.0003" iyz="0" izz="0.0004"/>
+    </inertial>
+  </link>
+  <link name="front_left_foot_link">
+    <visual>
+      <geometry>
+        <mesh filename="file://$(find quadruped_robot)/stl/lfoot.stl" scale="0.001 0.001 0.001"/>
+      </geometry>
+      <origin rpy="0 0 0" xyz="-0.120 0.04 0.1"/>
+      <material name="black">
+        <color rgba="0.0 0.0 0.0 1.0"/>
+      </material>
+    </visual>
+    <collision>
+      <geometry>
+        <mesh filename="file://$(find quadruped_robot)/stl/lfoot.stl" scale="0.001 0.001 0.001"/>
+      </geometry>
+      <origin rpy="0 0 0" xyz="-0.120 0.04 0.1"/>
+    </collision>
+    <inertial>
+      <mass value="0.1"/>
+      <inertia ixx="0.0001" ixy="0" ixz="0" iyy="0.0001" iyz="0" izz="0.0001"/>
+    </inertial>
+  </link>
+  <link name="front_left_toe_link">
+    <visual>
+      <geometry>
+        <mesh filename="file://$(find quadruped_robot)/stl/foot.stl" scale="0.001 0.001 0.001"/>
+      </geometry>
+      <origin rpy="0 -0.40010 0" xyz="0 -0.01 0"/>
+      <material name="grey">
+        <color rgba="0.6 0.6 0.6 1"/>
+      </material>
+    </visual>
+    <collision>
+      <geometry>
+        <mesh filename="file://$(find quadruped_robot)/stl/foot.stl" scale="0.001 0.001 0.001"/>
+      </geometry>
+      <origin rpy="0 -0.40010 0" xyz="0 -0.01 0"/>
+      <contact_coefficients mu="1.5"/>
+    </collision>
+    <inertial>
+      <mass value="0.05"/>
+      <inertia ixx="0.00005" ixy="0" ixz="0" iyy="0.00005" iyz="0" izz="0.00005"/>
+    </inertial>
+  </link>
+  <joint name="front_left_shoulder" type="revolute">
+    <parent link="base_link"/>
+    <child link="front_left_shoulder_link"/>
+    <axis xyz="1 0 0"/>
+    <origin rpy="0 0 0" xyz="-0.093 -0.036 0"/>
+    <limit effort="25" lower="-3.141592653589793" upper="3.141592653589793" velocity="1.5"/>
+    <dynamics damping="0.0" friction="0.5"/>
+  </joint>
+  <joint name="front_left_leg" type="revolute">
+    <parent link="front_left_shoulder_link"/>
+    <child link="front_left_leg_link"/>
+    <axis xyz="0 1 0"/>
+    <origin rpy="0 0 0" xyz="0 -0.052 0"/>
+    <limit effort="25" lower="-3.141592653589793" upper="3.141592653589793" velocity="1.5"/>
+    <dynamics damping="0.0" friction="0.0"/>
+  </joint>
+  <joint name="front_left_leg_cover_joint" type="fixed">
+    <parent link="front_left_leg_link"/>
+    <child link="front_left_leg_link_cover"/>
+    <origin xyz="0 0 0"/>
+  </joint>
+  <joint name="front_left_foot" type="revolute">
+    <parent link="front_left_leg_link"/>
+    <child link="front_left_foot_link"/>
+    <axis xyz="0 1 0"/>
+    <origin rpy="0 0 0" xyz="-0.01 0 -0.12"/>
+        <limit effort="25" lower="-3.141592653589793" upper="3.141592653589793" velocity="1.5"/>
+    <dynamics damping="0.0" friction="0.5"/>
+  </joint>
+  <joint name="front_left_toe" type="fixed">
+    <parent link="front_left_foot_link"/>
+    <child link="front_left_toe_link"/>
+    <origin xyz="0 0 -0.115"/>
+  </joint>
+  <link name="front_right_shoulder_link">
+    <visual>
+      <geometry>
+        <mesh filename="file://$(find quadruped_robot)/stl/rshoulder.stl" scale="0.001 0.001 0.001"/>
+      </geometry>
+      <origin rpy="0 0 0" xyz="-0.135 -0.09 -0.01"/>
+      <material name="black">
+        <color rgba="0.0 0.0 0.0 1.0"/>
+      </material>
+    </visual>
+    <collision>
+      <geometry>
+        <mesh filename="file://$(find quadruped_robot)/stl/rshoulder.stl" scale="0.001 0.001 0.001"/>
+      </geometry>
+      <origin rpy="0 0 0" xyz="-0.135 -0.09 -0.01"/>
+    </collision>
+    <inertial>
+      <mass value="0.30"/>
+      <inertia ixx="0.0005" ixy="0" ixz="0" iyy="0.0006" iyz="0" izz="0.0007"/>
+    </inertial>
+  </link>
+  <link name="front_right_leg_link_cover">
+    <visual>
+      <geometry>
+        <mesh filename="file://$(find quadruped_robot)/stl/rarm_cover.stl" scale="0.001 0.001 0.001"/>
+      </geometry>
+      <origin rpy="0 0 0" xyz="-0.125 -0.15 -0.02"/>
+      <material name="yellow">
+        <color rgba="0.92 0.83 0.0 1"/>
+      </material>
+    </visual>
+  </link>
+  <link name="front_right_leg_link">
+    <visual>
+      <geometry>
+        <mesh filename="file://$(find quadruped_robot)/stl/rarm.stl" scale="0.001 0.001 0.001"/>
+      </geometry>
+      <origin rpy="0 0 0" xyz="-0.125 -0.15 -0.02"/>
+      <material name="black">
+        <color rgba="0.0 0.0 0.0 1.0"/>
+      </material>
+    </visual>
+    <collision>
+      <geometry>
+        <mesh filename="file://$(find quadruped_robot)/stl/rarm.stl" scale="0.001 0.001 0.001"/>
+      </geometry>
+      <origin rpy="0 0 0" xyz="-0.125 -0.15 -0.02"/>
+    </collision>
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